File: boost-converter/boost-converter.kicad_pcb (KiCad board)
At the start: 2 copper layers, 18 parts, among them P1 CONN_02X01, P2 CONN_02X01, Q1 IRF730, Q2 BC547, U1 NE555

Commit message: Zmiana footprintu potencjometru
Parts:
- RV1: footprint Potentiometers:Potentiometer_Trimmer-EVM3E -> Potentiometers:Potentiometer_Triwood_RM-065
Changed lines of the file:
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@@
     (links 33)
     (no_connects 33)
-    (area 0 0 0 0)
+    (area 29.955 61.039999 114.355 100.115)
     (thickness 1.6)
     (drawings 0)
@@
     )
   )
-  (module Potentiometers:Potentiometer_Trimmer-EVM3E (layer F.Cu)
-    (at 68.58 69.85)
-    (descr http://www.comkey.in/sites/default/files/attachments/EVM3ESX50B15.pdf)
-    (tags "trimmer smd")
-    (attr smd)
-    (fp_text reference RV1 (at 0 3.835) (layer F.SilkS)
-      (effects (font (size 1 1) (thickness 0.15)))
-    )
-    (fp_text value 1k (at 0 -3.785) (layer F.Fab)
-      (effects (font (size 1 1) (thickness 0.15)))
-    )
-    (fp_line (start 1.778 -1.753) (end 1.778 0.533) (layer F.SilkS) (width 0.15))
-    (fp_line (start 1.27 -1.753) (end 1.778 -1.753) (layer F.SilkS) (width 0.15))
-    (fp_line (start -1.778 -1.753) (end -1.27 -1.753) (layer F.SilkS) (width 0.15))
-    (fp_line (start -1.778 0.533) (end -1.778 -1.753) (layer F.SilkS) (width 0.15))
-    (fp_line (start 2.2 2.45) (end -2.2 2.45) (layer F.CrtYd) (width 0.05))
-    (fp_line (start 2.2 -2.6) (end 2.2 2.45) (layer F.CrtYd) (width 0.05))
-    (fp_line (start -2.2 -2.6) (end 2.2 -2.6) (layer F.CrtYd) (width 0.05))
-    (fp_line (start -2.2 2.45) (end -2.2 -2.6) (layer F.CrtYd) (width 0.05))
-    (fp_line (start 0.9 1.375) (end 0.9 1.725) (layer F.Fab) (width 0.05))
-    (fp_line (start 1.55 1.375) (end 0.9 1.375) (layer F.Fab) (width 0.05))
-    (fp_line (start -0.9 1.325) (end -0.9 1.725) (layer F.Fab) (width 0.05))
-    (fp_line (start -1.55 1.325) (end -0.9 1.325) (layer F.Fab) (width 0.05))
-    (fp_line (start -0.25 -0.225) (end -0.25 -0.975) (layer F.Fab) (width 0.05))
-    (fp_line (start -1 -0.225) (end -0.25 -0.225) (layer F.Fab) (width 0.05))
-    (fp_line (start -1 0.275) (end -1 -0.225) (layer F.Fab) (width 0.05))
-    (fp_line (start -0.25 0.275) (end -1 0.275) (layer F.Fab) (width 0.05))
-    (fp_line (start -0.25 1.025) (end -0.25 0.275) (layer F.Fab) (width 0.05))
-    (fp_line (start 0.25 1.025) (end -0.25 1.025) (layer F.Fab) (width 0.05))
-    (fp_line (start 0.25 0.275) (end 0.25 1.025) (layer F.Fab) (width 0.05))
-    (fp_line (start 1 0.275) (end 0.25 0.275) (layer F.Fab) (width 0.05))
-    (fp_line (start 1 -0.225) (end 1 0.275) (layer F.Fab) (width 0.05))
-    (fp_line (start 0.25 -0.225) (end 1 -0.225) (layer F.Fab) (width 0.05))
-    (fp_line (start 0.25 -0.975) (end 0.25 -0.225) (layer F.Fab) (width 0.05))
-    (fp_line (start -0.25 -0.975) (end 0.25 -0.975) (layer F.Fab) (width 0.05))
-    (fp_line (start -1.55 1.725) (end -1.55 -1.525) (layer F.Fab) (width 0.05))
-    (fp_line (start 1.55 1.725) (end -1.55 1.725) (layer F.Fab) (width 0.05))
-    (fp_line (start 1.55 -1.525) (end 1.55 1.725) (layer F.Fab) (width 0.05))
-    (fp_line (start -1.55 -1.525) (end 1.55 -1.525) (layer F.Fab) (width 0.05))
-    (fp_circle (center 0 0.025) (end 0 -0.225) (layer F.Fab) (width 0.05))
-    (fp_circle (center 0 0.025) (end 0 -1.175) (layer F.Fab) (width 0.05))
-    (fp_circle (center 0 0.025) (end 0 -1.525) (layer F.Fab) (width 0.05))
-    (pad 1 smd rect (at -1.4 1.625) (size 1.2 1.2) (layers F.Cu F.Paste F.Mask)
-      (net 10 "Net-(R1-Pad2)"))
-    (pad 3 smd rect (at 1.4 1.625) (size 1.2 1.2) (layers F.Cu F.Paste F.Mask)
-      (net 11 "Net-(R2-Pad1)"))
-    (pad 2 smd rect (at 0 -1.625) (size 1.6 1.5) (layers F.Cu F.Paste F.Mask)
-      (net 8 "Net-(Q2-Pad2)"))
-  )
   (module Housings_DIP:DIP-8_W7.62mm_Socket_LongPads (layer F.Cu)
     (at 82.55 87.63 90)
@@
       (rotate (xyz 0 0 0))
     )
+  )
+  (module Potentiometers:Potentiometer_Triwood_RM-065 (layer F.Cu)
+    (at 68.58 69.85)
+    (descr "Potentiometer, Trimmer, RM-065")
+    (tags "Potentiometer, Trimmer, RM-065")
+    (fp_text reference RV1 (at 6.30936 -6.30936) (layer F.SilkS)
+      (effects (font (size 1 1) (thickness 0.15)))
+    )
+    (fp_text value 1k (at 2.49936 2.58064) (layer F.Fab)
+      (effects (font (size 1 1) (thickness 0.15)))
+    )
+    (fp_line (start 2.24536 -2.88036) (end 2.24536 -3.64236) (layer F.SilkS) (width 0.15))
+    (fp_line (start 2.75336 -2.88036) (end 2.75336 -3.64236) (layer F.SilkS) (width 0.15))
+    (fp_arc (start 2.49936 -2.49936) (end 4.15036 -2.24536) (angle 90) (layer F.SilkS) (width 0.15))
+    (fp_arc (start 2.49936 -2.49936) (end 2.62636 -0.84836) (angle 90) (layer F.SilkS) (width 0.15))
+    (fp_arc (start 2.49936 -2.49936) (end 3.38836 -3.89636) (angle 90) (layer F.SilkS) (width 0.15))
+    (fp_arc (start 2.49936 -2.49936) (end 1.10236 -1.61036) (angle 90) (layer F.SilkS) (width 0.15))
+    (fp_line (start -0.80264 1.31064) (end -0.80264 1.18364) (layer F.SilkS) (width 0.15))
+    (fp_line (start -0.80264 -2.49936) (end -0.80264 -1.10236) (layer F.SilkS) (width 0.15))
+    (fp_line (start 5.80136 1.31064) (end 5.80136 1.18364) (layer F.SilkS) (width 0.15))
+    (fp_line (start 5.80136 -2.49936) (end 5.80136 -1.10236) (layer F.SilkS) (width 0.15))
+    (fp_line (start 1.35636 0.42164) (end 1.73736 0.54864) (layer F.SilkS) (width 0.15))
+    (fp_line (start 1.73736 0.54864) (end 2.49936 0.67564) (layer F.SilkS) (width 0.15))
+    (fp_line (start 2.49936 0.67564) (end 3.26136 0.54864) (layer F.SilkS) (width 0.15))
+    (fp_line (start 3.26136 0.54864) (end 3.64236 0.42164) (layer F.SilkS) (width 0.15))
+    (fp_line (start 1.22936 -0.46736) (end 3.76936 -0.46736) (layer F.SilkS) (width 0.15))
+    (fp_arc (start 2.49936 -2.49936) (end 3.76936 -5.42036) (angle 90) (layer F.SilkS) (width 0.15))
+    (fp_arc (start 2.49936 -2.49936) (end -0.42164 -1.22936) (angle 90) (layer F.SilkS) (width 0.15))
+    (fp_line (start 4.53136 -5.80136) (end 3.64236 -5.80136) (layer F.SilkS) (width 0.15))
+    (fp_line (start 1.35636 -5.80136) (end 0.46736 -5.80136) (layer F.SilkS) (width 0.15))
+    (fp_line (start 4.15036 -2.88036) (end 4.65836 -2.88036) (layer F.SilkS) (width 0.15))
+    (fp_line (start 4.65836 -2.88036) (end 4.65836 -2.11836) (layer F.SilkS) (width 0.15))
+    (fp_line (start 4.65836 -2.11836) (end 4.15036 -2.11836) (layer F.SilkS) (width 0.15))
+    (fp_line (start 0.84836 -2.88036) (end 0.34036 -2.88036) (layer F.SilkS) (width 0.15))
+    (fp_line (start 0.34036 -2.88036) (end 0.34036 -2.11836) (layer F.SilkS) (width 0.15))
+    (fp_line (start 0.34036 -2.11836) (end 0.84836 -2.11836) (layer F.SilkS) (width 0.15))
+    (fp_line (start 3.00736 -2.24536) (end 4.15036 -2.24536) (layer F.SilkS) (width 0.15))
+    (fp_line (start 3.00736 -2.75336) (end 4.15036 -2.75336) (layer F.SilkS) (width 0.15))
+    (fp_line (start 1.99136 -2.24536) (end 0.84836 -2.24536) (layer F.SilkS) (width 0.15))
+    (fp_line (start 1.99136 -2.75336) (end 0.84836 -2.75336) (layer F.SilkS) (width 0.15))
+    (fp_line (start 2.75336 -2.11836) (end 2.75336 -0.84836) (layer F.SilkS) (width 0.15))
+    (fp_line (start 2.24536 -2.11836) (end 2.24536 -0.84836) (layer F.SilkS) (width 0.15))
+    (fp_line (start 1.99136 -2.88036) (end 1.99136 -2.11836) (layer F.SilkS) (width 0.15))
+    (fp_line (start 1.99136 -2.11836) (end 3.00736 -2.11836) (layer F.SilkS) (width 0.15))
+    (fp_line (start 3.00736 -2.11836) (end 3.00736 -2.88036) (layer F.SilkS) (width 0.15))
+    (fp_line (start 3.00736 -2.88036) (end 1.99136 -2.88036) (layer F.SilkS) (width 0.15))
+    (fp_line (start 0.46736 -5.80136) (end -0.80264 -4.40436) (layer F.SilkS) (width 0.15))
+    (fp_line (start -0.80264 -4.40436) (end -0.80264 -2.49936) (layer F.SilkS) (width 0.15))
+    (fp_line (start 4.53136 -5.80136) (end 5.80136 -4.40436) (layer F.SilkS) (width 0.15))
+    (fp_line (start 5.80136 -4.40436) (end 5.80136 -2.49936) (layer F.SilkS) (width 0.15))
+    (fp_line (start 5.54736 1.31064) (end 5.54736 1.56464) (layer F.SilkS) (width 0.15))
+    (fp_line (start 5.54736 1.56464) (end 4.40436 1.56464) (layer F.SilkS) (width 0.15))
+    (fp_line (start 4.40436 1.56464) (end 4.40436 1.31064) (layer F.SilkS) (width 0.15))
+    (fp_line (start -0.54864 1.31064) (end -0.54864 1.56464) (layer F.SilkS) (width 0.15))
+    (fp_line (start -0.54864 1.56464) (end 0.59436 1.56464) (layer F.SilkS) (width 0.15))
+    (fp_line (start 0.59436 1.56464) (end 0.59436 1.31064) (layer F.SilkS) (width 0.15))
+    (fp_line (start -0.80264 1.31064) (end 5.80136 1.31064) (layer F.SilkS) (width 0.15))
+    (pad 2 thru_hole circle (at 2.49936 -5.03936) (size 2.49936 2.49936) (drill 1.19888) (layers *.Cu *.Mask)
+      (net 8 "Net-(Q2-Pad2)"))
+    (pad 3 thru_hole circle (at 4.99872 0) (size 2.49936 2.49936) (drill 1.19888) (layers *.Cu *.Mask)
+      (net 11 "Net-(R2-Pad1)"))
+    (pad 1 thru_hole circle (at 0 0) (size 2.49936 2.49936) (drill 1.19888) (layers *.Cu *.Mask)
+      (net 10 "Net-(R1-Pad2)"))
+    (model Potentiometers.3dshapes/Potentiometer_Triwood_RM-065.wrl
+      (at (xyz 0 0 0))
+      (scale (xyz 4 4 4))
+      (rotate (xyz 0 0 0))
+    )

Commit message: Dokończone pcb + pdf
Parts:
- moved C4 17.3 mm to (102.9, 80.0), turned to 180 degrees
- moved C3 14.2 mm to (82.5, 92.7), turned to 180 degrees
- moved P1 13.5 mm to (97.8, 95.2), turned to 90 degrees
- moved Q1 12.0 mm to (59.7, 80.0)
- moved R1 8.98 mm to (47.0, 61.0)
- moved R3 7.18 mm to (53.3, 72.4)
- moved U1 5.68 mm to (77.5, 85.1)
- moved D1 5.08 mm to (48.3, 74.9)
- moved RV1 5.08 mm to (68.6, 64.8), turned to 270 degrees
- moved C1 4.58 mm to (49.5, 90.2), turned to 270 degrees
- moved R2 4.58 mm to (68.6, 74.9)
- moved R6 4.02 mm to (77.5, 73.7)
- moved R4 4.02 mm to (77.5, 63.5)
- moved Q2 3.59 mm to (92.7, 78.7)
- moved C2 2.54 mm to (58.4, 91.4), turned to 0 degrees
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Routing:
- net +9V: track 0.00 -> 164.0 mm
- net Earth: track 0.00 -> 121.3 mm
- net VSSA: track 0.00 -> 77.4 mm
- net Net-(C3-Pad1): track 0.00 -> 64.1 mm
- net Net-(D1-Pad2): track 0.00 -> 38.5 mm
- net Net-(Q2-Pad2): track 0.00 -> 32.3 mm
- net Net-(Q1-Pad3): track 0.00 -> 29.7 mm
- net Net-(R4-Pad2): track 0.00 -> 18.9 mm
- net Net-(Q2-Pad1): track 0.00 -> 12.0 mm
- net Net-(R1-Pad2): track 0.00 -> 10.5 mm
- net Net-(C2-Pad1): track 0.00 -> 8.45 mm
- net Net-(R2-Pad1): track 0.00 -> 5.16 mm
- added copper zone on F.Cu, net Earth
Other:
- board outline added: 78.7 x 44.4 mm
- net class Default: trace_width 0.25 -> 0.5
- rule trace_min: 0.2 -> 0.3
